File: design_revb_2chip/design_revb_2chip.kicad_sch (KiCad schematic)
At the start: 0 parts

Commit message: Initial Schematic Sheets
Created Initial Schematic Sheets and placed initial symbols for editing.
Other:
- added sheet ETH_SIDE (ETH_SIDE.kicad_sch)
- added sheet USB_SIDE (USB_SIDE.kicad_sch)
Changed lines of the file:
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@@
 	(generator_version "8.0")
 	(paper "A4")
+	(sheet
+		(at 158.75 31.75)
+		(size 113.03 113.03)
+		(fields_autoplaced yes)
+		(stroke
+			(width 0.1524)
+			(type solid)
+		)
+		(fill
+			(color 0 0 0 0.0000)
+		)
+		(property "Sheetname" "ETH_SIDE"
+			(at 158.75 31.0384 0)
+			(effects
+				(font
+					(size 1.27 1.27)
+				)
+				(justify left bottom)
+			)
+		)
+		(property "Sheetfile" "ETH_SIDE.kicad_sch"
+			(at 158.75 145.3646 0)
+			(effects
+				(font
+					(size 1.27 1.27)
+				)
+				(justify left top)
+			)
+		)
+		(instances
+			(project "design_revb_2chip"
+				(path "/d77d37fa-bfdc-44bb-83cc-90773a88d214"
+					(page "3")
+				)
+			)
+		)
+	)
+	(sheet
+		(at 19.05 22.86)
+		(size 104.14 128.27)
+		(fields_autoplaced yes)
+		(stroke
+			(width 0.1524)
+			(type solid)
+		)
+		(fill
+			(color 0 0 0 0.0000)
+		)
+		(property "Sheetname" "USB_SIDE"
+			(at 19.05 22.1484 0)
+			(effects
+				(font
+					(size 1.27 1.27)
+				)
+				(justify left bottom)
+			)
+		)
+		(property "Sheetfile" "USB_SIDE.kicad_sch"
+			(at 19.05 151.7146 0)
+			(effects
+				(font
+					(size 1.27 1.27)
+				)
+				(justify left top)
+			)
+		)
+		(instances
+			(project "design_revb_2chip"
+				(path "/d77d37fa-bfdc-44bb-83cc-90773a88d214"
+					(page "2")
+				)
+			)
+		)
+	)
 	(sheet_instances
 		(path "/"
