File: design_revb_2chip/ETH_SIDE.kicad_sch (KiCad schematic)
At the start: 50 parts, among them J3 09452812810, U4 DP83TG720SWRHARQ1, U5 TPS784105QWDRBRQ1, U6 219-5MST

Commit message: footprint resizing
Parts:
- C27, C28, C31, C35, C36, C37, C38, C39, C40, C41, C42, C43, C44, C46, C47, C48, C49, C50: footprint Capacitor_SMD:C_0201_0603Metric -> Capacitor_SMD:C_0402_1005Metric
- C29, C30, C32, C33, C34: footprint Capacitor_SMD:C_0201_0603Metric -> Capacitor_SMD:C_0603_1608Metric
- C45: footprint (none) -> Capacitor_SMD:C_0603_1608Metric
Changed lines of the file:
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@@
 			)
 		)
-		(property "Footprint" "Capacitor_SMD:C_0201_0603Metric"
+		(property "Footprint" "Capacitor_SMD:C_0402_1005Metric"
 			(at 267.0048 119.38 0)
 			(effects
@@
 			)
 		)
-		(property "Footprint" "Capacitor_SMD:C_0201_0603Metric"
+		(property "Footprint" "Capacitor_SMD:C_0402_1005Metric"
 			(at 276.5552 101.6 0)
 			(effects
@@
 			)
 		)
-		(property "Footprint" "Capacitor_SMD:C_0201_0603Metric"
+		(property "Footprint" "Capacitor_SMD:C_0402_1005Metric"
 			(at 52.07 96.8248 0)
 			(effects
@@
 			)
 		)
-		(property "Footprint" "Capacitor_SMD:C_0201_0603Metric"
+		(property "Footprint" "Capacitor_SMD:C_0603_1608Metric"
 			(at 190.1952 151.13 0)
 			(effects
@@
 			)
 		)
-		(property "Footprint" "Capacitor_SMD:C_0201_0603Metric"
+		(property "Footprint" "Capacitor_SMD:C_0402_1005Metric"
 			(at 238.4552 101.6 0)
 			(effects
@@
 			)
 		)
-		(property "Footprint" ""
+		(property "Footprint" "Capacitor_SMD:C_0603_1608Metric"
 			(at 254.3048 58.42 0)
 			(effects
@@
 			)
 		)
-		(property "Footprint" "Capacitor_SMD:C_0201_0603Metric"
+		(property "Footprint" "Capacitor_SMD:C_0402_1005Metric"
 			(at 200.3552 140.97 0)
 			(effects
@@
 			)
 		)
-		(property "Footprint" "Capacitor_SMD:C_0201_0603Metric"
+		(property "Footprint" "Capacitor_SMD:C_0402_1005Metric"
 			(at 270.2052 26.67 0)
 			(effects
@@
 			)
 		)
-		(property "Footprint" "Capacitor_SMD:C_0201_0603Metric"
+		(property "Footprint" "Capacitor_SMD:C_0402_1005Metric"
 			(at 238.4552 119.38 0)
 			(effects
@@
 			)
 		)
-		(property "Footprint" "Capacitor_SMD:C_0201_0603Metric"
+		(property "Footprint" "Capacitor_SMD:C_0402_1005Metric"
 			(at 200.3552 101.6 0)
 			(effects
@@
 			)
 		)
-		(property "Footprint" "Capacitor_SMD:C_0201_0603Metric"
+		(property "Footprint" "Capacitor_SMD:C_0402_1005Metric"
 			(at 240.9952 80.01 0)
 			(effects
@@
 			)
 		)
-		(property "Footprint" "Capacitor_SMD:C_0201_0603Metric"
+		(property "Footprint" "Capacitor_SMD:C_0402_1005Metric"
 			(at 225.7552 119.38 0)
 			(effects
@@
 			)
 		)
-		(property "Footprint" "Capacitor_SMD:C_0201_0603Metric"
+		(property "Footprint" "Capacitor_SMD:C_0603_1608Metric"
 			(at 220.6752 27.94 0)
 			(effects
@@
 			)
 		)
-		(property "Footprint" "Capacitor_SMD:C_0201_0603Metric"
+		(property "Footprint" "Capacitor_SMD:C_0603_1608Metric"
 			(at 55.5752 135.89 0)
 			(effects
@@
 			)
 		)
-		(property "Footprint" "Capacitor_SMD:C_0201_0603Metric"
+		(property "Footprint" "Capacitor_SMD:C_0402_1005Metric"
 			(at 44.45 108.9152 0)
 			(effects
@@
 			)
 		)
-		(property "Footprint" "Capacitor_SMD:C_0201_0603Metric"
+		(property "Footprint" "Capacitor_SMD:C_0402_1005Metric"
 			(at 200.3552 62.23 0)
 			(effects
@@
 			)
 		)
-		(property "Footprint" "Capacitor_SMD:C_0201_0603Metric"
+		(property "Footprint" "Capacitor_SMD:C_0603_1608Metric"
 			(at 190.1952 72.39 0)
 			(effects
@@
 			)
 		)
-		(property "Footprint" "Capacitor_SMD:C_0201_0603Metric"
+		(property "Footprint" "Capacitor_SMD:C_0603_1608Metric"
 			(at 207.9752 27.94 0)
 			(effects
@@
 			)
 		)
-		(property "Footprint" "Capacitor_SMD:C_0201_0603Metric"
+		(property "Footprint" "Capacitor_SMD:C_0402_1005Metric"
 			(at 138.1252 111.76 0)
 			(effects
@@
 			)
 		)
-		(property "Footprint" "Capacitor_SMD:C_0201_0603Metric"
+		(property "Footprint" "Capacitor_SMD:C_0402_1005Metric"
 			(at 225.7552 80.01 0)
 			(effects
@@
 			)
 		)
-		(property "Footprint" "Capacitor_SMD:C_0201_0603Metric"
+		(property "Footprint" "Capacitor_SMD:C_0402_1005Metric"
 			(at 238.4552 140.97 0)
 			(effects
@@
 			)
 		)
-		(property "Footprint" "Capacitor_SMD:C_0201_0603Metric"
+		(property "Footprint" "Capacitor_SMD:C_0402_1005Metric"
 			(at 238.4552 62.23 0)
 			(effects
@@
 			)
 		)
-		(property "Footprint" "Capacitor_SMD:C_0201_0603Metric"
+		(property "Footprint" "Capacitor_SMD:C_0402_1005Metric"
 			(at 190.1952 111.76 0)
 			(effects
@@
 			)
 		)
-		(property "Footprint" "Capacitor_SMD:C_0201_0603Metric"
+		(property "Footprint" "Capacitor_SMD:C_0402_1005Metric"
 			(at 276.5552 140.97 0)
 			(effects

Commit message: Final Push for Rev A 1.0
Parts:
- C30, C32, C34, C45: footprint Capacitor_SMD:C_0603_1608Metric -> Capacitor_SMD:C_0402_1005Metric
- C33: footprint Capacitor_SMD:C_0603_1608Metric -> Capacitor_SMD:C_0805_2012Metric
- C49: footprint Capacitor_SMD:C_0402_1005Metric -> Capacitor_SMD:C_0805_2012Metric
Changed lines of the file:
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@@
 	(label "LED_0_DIP"
 		(at 12.7 182.88 0)
+		(fields_autoplaced yes)
 		(effects
 			(font
@@
 	(label "LED_0_STRP_ON"
 		(at 85.09 153.67 0)
+		(fields_autoplaced yes)
 		(effects
 			(font
@@
 	(label "LED_1"
 		(at 85.09 176.53 0)
+		(fields_autoplaced yes)
 		(effects
 			(font
@@
 	(label "Vdda3p3"
 		(at 264.16 140.97 0)
+		(fields_autoplaced yes)
 		(effects
 			(font
@@
 	(label "Vdd1.0"
 		(at 181.61 104.14 0)
+		(fields_autoplaced yes)
 		(effects
 			(font
@@
 	(label "BI_DA+"
 		(at 39.37 97.79 0)
+		(fields_autoplaced yes)
 		(effects
 			(font
@@
 	(label "LED_0_STRP_OFF"
 		(at 67.31 182.88 0)
+		(fields_autoplaced yes)
 		(effects
 			(font
@@
 	(label "Vsleep"
 		(at 264.16 156.21 0)
+		(fields_autoplaced yes)
 		(effects
 			(font
@@
 	(label "RX_D1_DIP"
 		(at 12.7 177.8 0)
+		(fields_autoplaced yes)
 		(effects
 			(font
@@
 	(label "LED_1"
 		(at 27.94 43.18 0)
+		(fields_autoplaced yes)
 		(effects
 			(font
@@
 	(label "RX_D0_DIP"
 		(at 12.7 175.26 0)
+		(fields_autoplaced yes)
 		(effects
 			(font
@@
 	(label "TRD_P"
 		(at 27.94 58.42 0)
+		(fields_autoplaced yes)
 		(effects
 			(font
@@
 	(label "TRD_P"
 		(at 15.24 97.79 0)
+		(fields_autoplaced yes)
 		(effects
 			(font
@@
 	(label "RX_D0_STRP"
 		(at 67.31 175.26 0)
+		(fields_autoplaced yes)
 		(effects
 			(font
@@
 	(label "BI_DA-"
 		(at 77.47 102.87 0)
+		(fields_autoplaced yes)
 		(effects
 			(font
@@
 	(label "BI_DA+"
 		(at 77.47 100.33 0)
+		(fields_autoplaced yes)
 		(effects
 			(font
@@
 	(label "RX_D2_DIP"
 		(at 12.7 180.34 0)
+		(fields_autoplaced yes)
 		(effects
 			(font
@@
 	(label "LED_0_DIP"
 		(at 12.7 185.42 0)
+		(fields_autoplaced yes)
 		(effects
 			(font
@@
 	(label "VddioB"
 		(at 81.28 38.1 0)
+		(fields_autoplaced yes)
 		(effects
 			(font
@@
 	(label "RX_D2_STRP"
 		(at 67.31 180.34 0)
+		(fields_autoplaced yes)
 		(effects
 			(font
@@
 	(label "TRD_N"
 		(at 15.24 107.95 0)
+		(fields_autoplaced yes)
 		(effects
 			(font
@@
 	(label "RX_D2_DIP"
 		(at 100.33 63.5 0)
+		(fields_autoplaced yes)
 		(effects
 			(font
@@
 	(label "Vdd1p0B"
 		(at 264.16 111.76 0)
+		(fields_autoplaced yes)
 		(effects
 			(font
@@
 	(label "Vdd1p0A"
 		(at 264.16 93.98 0)
+		(fields_autoplaced yes)
 		(effects
 			(font
@@
 	(label "VddioB"
 		(at 259.08 72.39 0)
+		(fields_autoplaced yes)
 		(effects
 			(font
@@
 	(label "RX_D1_STRP"
 		(at 130.81 33.02 0)
+		(fields_autoplaced yes)
 		(effects
 			(font
@@
 	(label "BI_DA-"
 		(at 39.37 107.95 0)
+		(fields_autoplaced yes)
 		(effects
 			(font
@@
 	(label "TRD_N"
 		(at 27.94 60.96 0)
+		(fields_autoplaced yes)
 		(effects
 			(font
@@
 	(label "LED_0_DIP"
 		(at 100.33 35.56 0)
+		(fields_autoplaced yes)
 		(effects
 			(font
@@
 	(label "Vsleep"
 		(at 27.94 45.72 0)
+		(fields_autoplaced yes)
 		(effects
 			(font
@@
 	(label "LED_0_STRP_ON"
 		(at 67.31 185.42 0)
+		(fields_autoplaced yes)
 		(effects
 			(font
@@
 	(label "Vdd1p0B"
 		(at 81.28 72.39 0)
+		(fields_autoplaced yes)
 		(effects
 			(font
@@
 	(label "LED_0_STRP_OFF"
 		(at 85.09 132.08 0)
+		(fields_autoplaced yes)
 		(effects
 			(font
@@
 	(label "Vdd1.0"
 		(at 275.59 27.94 0)
+		(fields_autoplaced yes)
 		(effects
 			(font
@@
 	(label "Vdda3p3"
 		(at 27.94 55.88 0)
+		(fields_autoplaced yes)
 		(effects
 			(font
@@
 	(label "RX_D1_DIP"
 		(at 100.33 54.61 0)
+		(fields_autoplaced yes)
 		(effects
 			(font
@@
 	(label "RX_D0_DIP"
 		(at 100.33 44.45 0)
+		(fields_autoplaced yes)
 		(effects
 			(font
@@
 	(label "RX_D2_STRP"
 		(at 130.81 41.91 0)
+		(fields_autoplaced yes)
 		(effects
 			(font
@@
 	(label "Vdd1p0A"
 		(at 27.94 50.8 0)
+		(fields_autoplaced yes)
 		(effects
 			(font
@@
 	(label "VddioA"
 		(at 87.63 69.85 180)
+		(fields_autoplaced yes)
 		(effects
 			(font
@@
 	(label "VddioA"
 		(at 259.08 55.88 0)
+		(fields_autoplaced yes)
 		(effects
 			(font
@@
 	(label "RX_D0_STRP"
 		(at 130.81 24.13 0)
+		(fields_autoplaced yes)
 		(effects
 			(font
@@
 	(label "RX_D1_STRP"
 		(at 67.31 177.8 0)
+		(fields_autoplaced yes)
 		(effects
 			(font
@@
 			)
 		)
-		(property "Footprint" "Capacitor_SMD:C_0603_1608Metric"
+		(property "Footprint" "Capacitor_SMD:C_0402_1005Metric"
 			(at 190.1952 151.13 0)
 			(effects
@@
 			)
 		)
-		(property "Footprint" "Capacitor_SMD:C_0603_1608Metric"
+		(property "Footprint" "Capacitor_SMD:C_0402_1005Metric"
 			(at 254.3048 58.42 0)
 			(effects
@@
 			)
 		)
-		(property "Footprint" "Capacitor_SMD:C_0402_1005Metric"
+		(property "Footprint" "Capacitor_SMD:C_0805_2012Metric"
 			(at 270.2052 26.67 0)
 			(effects
@@
 			)
 		)
-		(property "Footprint" "Capacitor_SMD:C_0603_1608Metric"
+		(property "Footprint" "Capacitor_SMD:C_0402_1005Metric"
 			(at 220.6752 27.94 0)
 			(effects
@@
 			)
 		)
-		(property "Footprint" "Capacitor_SMD:C_0603_1608Metric"
+		(property "Footprint" "Capacitor_SMD:C_0402_1005Metric"
 			(at 190.1952 72.39 0)
 			(effects
@@
 			)
 		)
-		(property "Footprint" "Capacitor_SMD:C_0603_1608Metric"
+		(property "Footprint" "Capacitor_SMD:C_0805_2012Metric"
 			(at 207.9752 27.94 0)
 			(effects
